File: branches/v1/wrt54_relay_board.brd (EAGLE design)
At the start: 90.5 x 87 mm, 61 parts, among them IC1 18F2550, IC2 786TV, IC3 MAX232, K1 351, K2 351, T1 2STX1360, T2 2STX1360, X1 C-GRID-05-70543

Commit message: added missing resistor between wrt54-tx and pic-rx - it burned the tx port twice :-(
added flush command to delete all rfid
Parts:
- added R11: 10k, resistor:0204V
Connections:
- new net N$39: JP5.3, R11.2
- net N$25: now also R11.1; no longer JP5.3
Routing:
- net N$25: track 28.2 -> 19.4 mm
- net N$39: track 0.00 -> 6.35 mm
Changed lines of the file:
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@@
 <element name="C7" library="capacitor-wima" package="C5B2.5" value="100nF" x="74.93" y="26.035" rot="R90"/>
 <element name="C8" library="capacitor-wima" package="C5B2.5" value="100nF" x="78.74" y="31.115" rot="R180"/>
+<element name="R11" library="resistor" package="0204V" value="10k" x="12.7" y="17.78" rot="R180"/>
 </elements>
 <signals>
@@
 <wire x1="23.495" y1="23.495" x2="26.67" y2="23.495" width="1.016" layer="16"/>
 <wire x1="37.465" y1="23.495" x2="34.29" y2="23.495" width="1.016" layer="16"/>
-<wire x1="26.67" y1="23.495" x2="34.29" y2="23.495" width="0" layer="19" extent="16-16"/>
 <via x="26.67" y="23.495" extent="1-16" drill="0.6" diameter="1.6764"/>
 <via x="34.29" y="23.495" extent="1-16" drill="0.6" diameter="1.6764"/>
+<wire x1="26.67" y1="23.495" x2="34.29" y2="23.495" width="0" layer="19" extent="1-1"/>
 </signal>
 <signal name="N$16">
@@
 <signal name="N$25">
 <contactref element="IC1" pad="18"/>
-<contactref element="JP5" pad="3"/>
 <wire x1="16.51" y1="31.75" x2="19.05" y2="31.75" width="1.016" layer="16"/>
 <wire x1="19.05" y1="31.75" x2="19.05" y2="21.59" width="1.016" layer="16"/>
 <wire x1="19.05" y1="21.59" x2="15.24" y2="17.78" width="1.016" layer="16"/>
-<wire x1="15.24" y1="17.78" x2="5.08" y2="17.78" width="1.016" layer="16"/>
+<contactref element="R11" pad="1"/>
+<wire x1="15.24" y1="17.78" x2="13.97" y2="17.78" width="1.016" layer="16"/>
 </signal>
 <signal name="N$26">
@@
 <wire x1="78.105" y1="8.255" x2="84.7725" y2="8.255" width="0.6096" layer="16"/>
 <wire x1="84.7725" y1="8.255" x2="85.09" y2="8.5725" width="0.6096" layer="16"/>
-<wire x1="81.28" y1="34.925" x2="81.28" y2="31.115" width="0" layer="19" extent="16-16"/>
 <via x="20.955" y="27.305" extent="1-16" drill="0.6" diameter="1.6764"/>
 <wire x1="26.67" y1="27.305" x2="24.765" y2="27.305" width="1.016" layer="16"/>
-<wire x1="24.765" y1="27.305" x2="20.955" y2="27.305" width="0" layer="19" extent="1-16"/>
+<wire x1="81.28" y1="34.925" x2="81.28" y2="31.115" width="0" layer="19" extent="16-16"/>
+<wire x1="20.955" y1="27.305" x2="24.765" y2="27.305" width="0" layer="19" extent="16-16"/>
 </signal>
 <signal name="N$28">
@@
 <via x="24.765" y="27.305" extent="1-16" drill="0.6" diameter="1.6764"/>
 </signal>
+<signal name="N$39">
+<contactref element="JP5" pad="3"/>
+<contactref element="R11" pad="2"/>
+<wire x1="11.43" y1="17.78" x2="5.08" y2="17.78" width="1.016" layer="16"/>
+</signal>
 </signals>
-<errors>
-</errors>
 </board>
 </drawing>
